File: TrlBoard.kicad_pcb (KiCad board)
At the start: 2 copper layers, 56.5 x 27.9 mm, 49 parts, among them J1 B2B-XH-A_LF__SN_, J2 Conn_01x22, J4 Conn_01x22, J5 USB_C_Receptacle_USB2.0_16P, Q1 SS8050-G, Q2 SS8050-G, U1 BQ24072RGT, U2 ESP32-S3-WROOM-1, U3 TPS63060, U4 CH340C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

Commit message: ICM + Update cost
Parts:
- removed C17: 100nF, Capacitor_SMD:C_0402_1005Metric
- removed C18: 2.2nF, Capacitor_SMD:C_0402_1005Metric
- removed R15: 10k, Resistor_SMD:R_0402_1005Metric
- removed U5: MPU-6050, Sensor_Motion:InvenSense_QFN-24_4x4mm_P0.5mm
- added C13: 10nF, Capacitor_SMD:C_0402_1005Metric, F.Cu at (157.8, 77.5)
- added MT1: ICM-42670-P, ICM-42670-P:XDCR_ICM-42670-P, F.Cu at (159.2, 73.2)
- C12: footprint Capacitor_SMD:C_0402_1005Metric -> Capacitor_SMD:C_0603_1608Metric
- C15: value 10uF -> 100nF
- C16: value 100nF -> 2.2uF
- C7, C8: footprint Capacitor_SMD:C_0603_1608Metric -> Capacitor_SMD:C_0402_1005Metric
- R2: value 111k -> 110k
- R3: footprint Resistor_SMD:R_0402_1005Metric -> Resistor_SMD:R_0603_1608Metric
- moved R14 2.47 mm to (157.2, 76.0), turned to -90 degrees
- moved C15 1.25 mm to (160.2, 77.5), turned to 0 degrees
- moved C16 1.25 mm to (160.2, 78.8), turned to 0 degrees
- moved G*** 0.75 mm to (149.2, 73.0)
- moved C3 0.50 mm to (179.8, 66.3)
- moved C4 0.50 mm to (171.0, 63.5)
- moved R4 0.50 mm to (179.8, 64.2)
- moved R6 0.50 mm to (179.8, 65.2)
- moved G*** 0.35 mm to (171.8, 75.0)
Connections:
- C15 pad 1: GND -> +3.3V
- C15 pad 2: +3.3V -> GND
- C16 pad 1: GND -> +3.3V
- C16 pad 2: +3.3V -> GND
- J4 pad 17: /GPIO13 -> VCC
- J4 pad 19: VCC -> +3.3V
- J4 pad 20: +3.3V -> GND
- R14 pad 1: +3.3V -> Net-(MT1-INT1/INT)
- R14 pad 2: /GPIO9 -> /GPIO11
Routing:
- net /GPIO13: track 27.6 -> 10.4 mm, vias 1 -> 2
- net /RXD0: track 27.9 -> 39.7 mm
- net Net-(U5-CPOUT): track 5.69 -> 0.00 mm
- net /GPIO9: track 16.9 -> 12.4 mm
- net Net-(U5-REGOUT): track 4.36 -> 0.00 mm
- net /GPIO10: track 17.0 -> 12.8 mm
- net +3.3V: track 138.9 -> 134.9 mm, vias 6 -> 4
- net Net-(MT1-INT1/INT): track 0.00 -> 2.18 mm
- net Net-(C4-Pad1): track 15.6 -> 17.2 mm
- net Net-(U3-VAUX): track 1.25 -> 0.00 mm
- net VCC: track 88.9 -> 88.0 mm
- net /GPIO11: track 4.92 -> 4.14 mm, vias 2 -> 0
- net /GPIO12: track 5.04 -> 5.31 mm, vias 2 -> 0
Other:
- board text removed: "R3"
