File: TrlBoard.kicad_sch (KiCad schematic)
At the start: 46 parts, among them J1 B2B-XH-A_LF__SN_, J2 Conn_01x22, J4 Conn_01x22, J5 USB_C_Receptacle_USB2.0_16P, Q1 SS8050-G, Q2 SS8050-G, U1 BQ24072RGT, U2 ESP32-S3-WROOM-1, U3 TPS63060, U4 CH340C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

Commit message: ICM + Update cost
Parts:
- removed C17: 100nF, Capacitor_SMD:C_0402_1005Metric, symbol Device:C
- removed C18: 2.2nF, Capacitor_SMD:C_0402_1005Metric, symbol Device:C
- removed R15: 10k, Resistor_SMD:R_0402_1005Metric, symbol Device:R
- removed U5: MPU-6050, Sensor_Motion:InvenSense_QFN-24_4x4mm_P0.5mm, symbol Sensor_Motion:MPU-6050
- added C13: 10nF, Capacitor_SMD:C_0402_1005Metric, symbol Device:C
- added MT1: ICM-42670-P, ICM-42670-P:XDCR_ICM-42670-P, symbol ICM-42670-P:ICM-42670-P
- C12: footprint Capacitor_SMD:C_0402_1005Metric -> Capacitor_SMD:C_0603_1608Metric
- C15: value 10uF -> 100nF
- C16: value 100nF -> 2.2uF
- C7, C8: footprint Capacitor_SMD:C_0603_1608Metric -> Capacitor_SMD:C_0402_1005Metric
- R2: value 111k -> 110k
- R3: footprint Resistor_SMD:R_0402_1005Metric -> Resistor_SMD:R_0603_1608Metric
Connections:
- net +3.3V: now also C15.1, C16.1, J4.19 (Pin_19), C13.1, MT1.5 (VDDIO), MT1.8 (VDD); no longer C15.2, C16.2, J4.20 (Pin_20), R14.1
- net GND: now also C15.2, C16.2, J4.20 (Pin_20), C13.2, MT1.6 (GND), MT1.7 (FSYNC); no longer C15.1, C16.1
- net GPIO10: now also MT1.13 (AP_SCL/AP_SCLK)
- net GPIO11: now also R14.2
- net GPIO12: now also MT1.1 (AP_SDO/AP_AD0)
- net GPIO13: now also MT1.12 (AP_CS); no longer J4.17 (Pin_17)
- net GPIO9: now also MT1.14 (AP_SDA/AP_SDIO/AP_SDI); no longer R14.2
- net VCC: now also J4.17 (Pin_17); no longer J4.19 (Pin_19)
- new net: MT1.10 (RESV), MT1.11 (RESV), MT1.2 (RESV), MT1.3 (RESV)
- new net: MT1.4 (INT1/INT), R14.1
Other:
- note added: "ESP32-S3-WROOM-1"
- note added: "TRLBOARD"
- note added: "sensor"
- note removed: "sensors"
- moved on the sheet: J2, J4, U2
